File: hardware/carrier/carrier_proto.kicad_pcb (KiCad board)
At the start: 2 copper layers, 90 x 70 mm, 18 parts

Commit message: Carrier board: every guess into modules.csv, plus three real checks
Makes measurement the only remaining step. pinmap.csv is the electrical
truth; modules.csv now holds every physical guess (pin counts, pin order,
body outlines, confidence) so measuring a module is one row edit and a
re-run. gen_proto.py refuses to run on an unknown function name or a pin
count that disagrees with its footprint, and prints NOT READY TO BUILD while
any row is still GUESSED.

Three project-specific checks, each negative-tested by breaking the design:

- fw_pinmap_check.py reads hw_config.h and fails if any of the 18 signals
  drifts from pinmap.csv. Without it a firmware pin change leaves the layout,
  wire list and build sheet all self-consistent and all wrong.
- body_check.py compares module BODY rectangles, which pad-level checks and
  KiCad's courtyard DRC both miss. It found 7 collisions the pad view hid -
  the SD breakout overlapped the Pico by 18x23 mm and PS/2 and VGA hung off
  the board - which is what drove SD, VGA, PS/2 and the OLED off-board.
- grid_check.py keeps every pad on a protoboard hole.

MEASURE.md is the hand-off: what to measure per module, which two decisions
I defaulted and why, and how to reverse them.

Co-Authored-By: Claude Opus 5 <noreply@anthropic.com>
Claude-Session: https://claude.ai/code/session_017HNT3cC7Xc7tuBcwupyw7Q
Parts:
- J_LVL_HV: value BSS138 HV -> BSS138 4ch level converter -
- J_LVL_LV: value BSS138 LV -> BSS138 4ch level converter -
- J_OLED: value OLED G V SCL SDA -> SSD1306 128x64 0.96in
- J_PS2: value PS/2 D CLK 5V G -> PS/2 socket breakout
- J_SD: value SD CS SCK MOSI MISO V G -> microSD SPI breakout
- J_VGA: value VGA VS HS R G B GND -> Serial Wombat PCB_0024 VGA b
- TB1: value PWR IN 5V 3V3 GND -> 3-way screw terminal 2.54mm
- U_RAM1: value PSRAM 1 -> PSRAM APS6404L on DIP-8 adap
- U_RAM2: value PSRAM 2 -> PSRAM APS6404L on DIP-8 adap
